Commit message: Update URDF joint naming

File: assets/mistletoe_urdf/mistletoe_description/urdf/mistletoe.urdf (robot description, URDF)
Before this commit: robot mistletoe, 13 links, 12 joints
Joints:
- removed joint Revolute 11
- removed joint Revolute 12
- removed joint Revolute 15
- removed joint Revolute 16
- removed joint Revolute 17
- removed joint Revolute 18
- removed joint Revolute 20
- removed joint Revolute 21
- removed joint Revolute 22
- removed joint Revolute 23
- removed joint Revolute 24
- removed joint Revolute 25
- added joint HAA1: type continuous, parent base_link, child Hip_3, origin xyz=-0.389589 0.0 0.025 rpy=0 0 0, axis 1.0 0.0 -0.0
- added joint HAA2: type continuous, parent base_link, child Hip_4, origin xyz=-0.389589 0.243608 0.025 rpy=0 0 0, axis 1.0 0.0 -0.0
- added joint HAA3: type continuous, parent base_link, child Hip_1, origin xyz=0.255776 0.0 0.025 rpy=0 0 0, axis -1.0 0.0 0.0
- added joint HAA4: type continuous, parent base_link, child Hip_2, origin xyz=0.255776 0.243608 0.025 rpy=0 0 0, axis 1.0 0.0 -0.0
- added joint HFE1: type continuous, parent Hip_3, child ACTUATOR_V2.1__KNEE__v10_3, origin xyz=0.077906 -0.025 0.0 rpy=0 0 0, axis -0.0 1.0 -0.0
- added joint HFE2: type continuous, parent Hip_4, child ACTUATOR_V2.1__KNEE__v10_4, origin xyz=0.077906 0.025 0.0 rpy=0 0 0, axis -0.0 -1.0 -0.0
- added joint HFE3: type continuous, parent Hip_1, child ACTUATOR_V2.1__KNEE__v10_1, origin xyz=-0.077906 -0.025 0.0 rpy=0 0 0, axis 0.0 1.0 -0.0
- added joint HFE4: type continuous, parent Hip_2, child ACTUATOR_V2.1__KNEE__v10_2, origin xyz=-0.077906 0.025 0.0 rpy=0 0 0, axis 0.0 -1.0 0.0
- added joint KFE1: type continuous, parent ACTUATOR_V2.1__KNEE__v10_3, child ANKLE_v4_4, origin xyz=0.17587 -0.0445 0.0 rpy=0 0 0, axis -0.0 -1.0 0.0
- added joint KFE2: type continuous, parent ACTUATOR_V2.1__KNEE__v10_4, child ANKLE_v4_3, origin xyz=0.17587 0.0445 0.0 rpy=0 0 0, axis -0.0 1.0 0.0
- added joint KFE3: type continuous, parent ACTUATOR_V2.1__KNEE__v10_1, child ANKLE_v4_1, origin xyz=-0.17587 -0.0445 0.0 rpy=0 0 0, axis 0.0 -1.0 0.0
- added joint KFE4: type continuous, parent ACTUATOR_V2.1__KNEE__v10_2, child ANKLE_v4_2, origin xyz=-0.17587 0.0445 0.0 rpy=0 0 0, axis 0.0 1.0 -0.0

Commit message: Somewhat working configs

File: assets/mistletoe_urdf/mistletoe_description/urdf/mistletoe.urdf (robot description, URDF)
Before this commit: robot mistletoe, 13 links, 12 joints
Links:
- removed link ACTUATOR_V2.1__KNEE__v10_1
- removed link ACTUATOR_V2.1__KNEE__v10_2
- removed link ACTUATOR_V2.1__KNEE__v10_3
- removed link ACTUATOR_V2.1__KNEE__v10_4
- removed link ANKLE_v4_1
- removed link ANKLE_v4_2
- removed link ANKLE_v4_3
- removed link ANKLE_v4_4
- removed link base_link
- added link LEG_1_FOOT, mass 0.0707595437253254; collision mesh filename=package://mistletoe_description/meshes/ANKLE_v4_1.stl scale=0.001 0.001 0.001; visual mesh filename=package://mistletoe_description/meshes/ANKLE_v4_1.stl scale=0.001 0.001 0.001
- added link LEG_1_THIGH, mass 0.6687419456686833; collision mesh filename=package://mistletoe_description/meshes/ACTUATOR_V2.1__KNEE_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 scale=0.001 0.001 0.001; visual mesh filename=package://mistletoe_description/meshes/ACTUATOR_V2.1__KNEE_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 scale=0.001 0.001 0.001
- added link LEG_2_FOOT, mass 0.0707595437253254; collision mesh filename=package://mistletoe_description/meshes/ANKLE_v4_2.stl scale=0.001 0.001 0.001; visual mesh filename=package://mistletoe_description/meshes/ANKLE_v4_2.stl scale=0.001 0.001 0.001
- added link LEG_2_THIGH, mass 0.6687419456686833; collision mesh filename=package://mistletoe_description/meshes/ACTUATOR_V2.1__KNEE_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 scale=0.001 0.001 0.001; visual mesh filename=package://mistletoe_description/meshes/ACTUATOR_V2.1__KNEE_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 scale=0.001 0.001 0.001
- added link LEG_3_FOOT, mass 0.0707595437253254; collision mesh filename=package://mistletoe_description/meshes/ANKLE_v4_3.stl scale=0.001 0.001 0.001; visual mesh filename=package://mistletoe_description/meshes/ANKLE_v4_3.stl scale=0.001 0.001 0.001
- added link LEG_3_THIGH, mass 0.6687419456686833; collision mesh filename=package://mistletoe_description/meshes/ACTUATOR_V2.1__KNEE_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 scale=0.001 0.001 0.001; visual mesh filename=package://mistletoe_description/meshes/ACTUATOR_V2.1__KNEE_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 scale=0.001 0.001 0.001
- added link LEG_4_FOOT, mass 0.0707595437253254; collision mesh filename=package://mistletoe_description/meshes/ANKLE_v4_4.stl scale=0.001 0.001 0.001; visual mesh filename=package://mistletoe_description/meshes/ANKLE_v4_4.stl scale=0.001 0.001 0.001
- added link LEG_4_THIGH, mass 0.6687419456686833; collision mesh filename=package://mistletoe_description/meshes/ACTUATOR_V2.1__KNEE_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 scale=0.001 0.001 0.001; visual mesh filename=package://mistletoe_description/meshes/ACTUATOR_V2.1__KNEE_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 scale=0.001 0.001 0.001
- added link base, mass 2.781822888066483; collision mesh filename=package://mistletoe_description/meshes/base_link.stl scale=0.001 0.001 0.001; visual mesh filename=package://mistletoe_description/meshes/base_link.stl scale=0.001 0.001 0.001
Joints:
- removed joint HAA1
- removed joint HAA2
- removed joint HAA3
- removed joint HAA4
- removed joint HFE1
- removed joint HFE2
- removed joint HFE3
- removed joint HFE4
- removed joint KFE1
- removed joint KFE2
- removed joint KFE3
- removed joint KFE4
- added joint LEG_1_HAA: type continuous, parent base, child Hip_3, origin xyz=-0.389589 0.0 0.025 rpy=0 0 0, axis 1.0 0.0 -0.0
- added joint LEG_1_HFE: type continuous, parent Hip_3, child LEG_3_THIGH, origin xyz=0.077906 -0.025 0.0 rpy=0 0 0, axis -0.0 1.0 -0.0
- added joint LEG_1_KFE: type continuous, parent LEG_3_THIGH, child LEG_4_FOOT, origin xyz=0.17587 -0.0445 0.0 rpy=0 0 0, axis -0.0 -1.0 0.0
- added joint LEG_2_HAA: type continuous, parent base, child Hip_4, origin xyz=-0.389589 0.243608 0.025 rpy=0 0 0, axis 1.0 0.0 -0.0
- added joint LEG_2_HFE: type continuous, parent Hip_4, child LEG_4_THIGH, origin xyz=0.077906 0.025 0.0 rpy=0 0 0, axis -0.0 -1.0 -0.0
- added joint LEG_2_KFE: type continuous, parent LEG_4_THIGH, child LEG_3_FOOT, origin xyz=0.17587 0.0445 0.0 rpy=0 0 0, axis -0.0 1.0 0.0
- added joint LEG_3_HAA: type continuous, parent base, child Hip_1, origin xyz=0.255776 0.0 0.025 rpy=0 0 0, axis -1.0 0.0 0.0
- added joint LEG_3_HFE: type continuous, parent Hip_1, child LEG_1_THIGH, origin xyz=-0.077906 -0.025 0.0 rpy=0 0 0, axis 0.0 1.0 -0.0
- added joint LEG_3_KFE: type continuous, parent LEG_1_THIGH, child LEG_1_FOOT, origin xyz=-0.17587 -0.0445 0.0 rpy=0 0 0, axis 0.0 -1.0 0.0
- added joint LEG_4_HAA: type continuous, parent base, child Hip_2, origin xyz=0.255776 0.243608 0.025 rpy=0 0 0, axis 1.0 0.0 -0.0
- added joint LEG_4_HFE: type continuous, parent Hip_2, child LEG_2_THIGH, origin xyz=-0.077906 0.025 0.0 rpy=0 0 0, axis 0.0 -1.0 0.0
- added joint LEG_4_KFE: type continuous, parent LEG_2_THIGH, child LEG_2_FOOT, origin xyz=-0.17587 0.0445 0.0 rpy=0 0 0, axis 0.0 1.0 -0.0
